File: KiCad/esp32/esp32.kicad_sch (KiCad schematic)
At the start: 26 parts, among them J1 6130XX11121_61302211121, J2 6130XX11121_61302211121, J3 USB4105-GF-A, U1 ESP32-S3-MINI-1-N8, U2 COM-16347, U3 TLV75801PDRVR, U4 ENS210-LQFM, U5 D3V3XA4B10LP

Commit message: schemated complete erc pass
Parts:
- Boot1, Reset1: footprint (none) -> Button_Switch_THT:SW_TH_Tactile_Omron_B3F-100x
- C1, C2, C3, C4, C7: footprint (none) -> Capacitor_SMD:C_0603_1608Metric
- J1, J2: footprint 6130XX11121_61302211121:61302211121 -> Footprint:61302211121
- J3: footprint USB4105-GF-A:GCT_USB4105-GF-A -> Footprint:GCT_USB4105-GF-A
- R1, R2, R3, R4, R5: footprint (none) -> Resistor_SMD:R_0603_1608Metric
- U4: footprint ENS210-LQFM:XDCR_ENS210-LQFM -> Footprint:XDCR_ENS210-LQFM
Changed lines of the file:
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@@
 			)
 		)
-		(property "Footprint" ""
+		(property "Footprint" "Resistor_SMD:R_0603_1608Metric"
 			(at 70.358 91.44 90)
 			(effects
@@
 			)
 		)
-		(property "Footprint" ""
+		(property "Footprint" "Capacitor_SMD:C_0603_1608Metric"
 			(at 79.7052 78.74 0)
 			(effects
@@
 			)
 		)
-		(property "Footprint" ""
+		(property "Footprint" "Resistor_SMD:R_0603_1608Metric"
 			(at 73.152 38.1 90)
 			(effects
@@
 			)
 		)
-		(property "Footprint" ""
+		(property "Footprint" "Capacitor_SMD:C_0603_1608Metric"
 			(at 75.8952 53.34 0)
 			(effects
@@
 			)
 		)
-		(property "Footprint" "ENS210-LQFM:XDCR_ENS210-LQFM"
+		(property "Footprint" "Footprint:XDCR_ENS210-LQFM"
 			(at 245.11 30.48 0)
 			(effects
@@
 			)
 		)
-		(property "Footprint" ""
+		(property "Footprint" "Resistor_SMD:R_0603_1608Metric"
 			(at 183.642 107.95 90)
 			(effects
@@
 			)
 		)
-		(property "Footprint" "6130XX11121_61302211121:61302211121"
+		(property "Footprint" "Footprint:61302211121"
 			(at 54.61 162.56 0)
 			(effects
@@
 			)
 		)
-		(property "Footprint" ""
+		(property "Footprint" "Resistor_SMD:R_0603_1608Metric"
 			(at 74.422 91.44 90)
 			(effects
@@
 			)
 		)
-		(property "Footprint" "USB4105-GF-A:GCT_USB4105-GF-A"
+		(property "Footprint" "Footprint:GCT_USB4105-GF-A"
 			(at 215.9 123.19 0)
 			(effects
@@
 			)
 		)
-		(property "Footprint" "6130XX11121_61302211121:61302211121"
+		(property "Footprint" "Footprint:61302211121"
 			(at 71.12 162.56 0)
 			(effects
@@
 			)
 		)
-		(property "Footprint" ""
+		(property "Footprint" "Capacitor_SMD:C_0603_1608Metric"
 			(at 141.9352 49.53 0)
 			(effects
@@
 			)
 		)
-		(property "Footprint" ""
+		(property "Footprint" "Button_Switch_THT:SW_TH_Tactile_Omron_B3F-100x"
 			(at 66.04 64.77 0)
 			(effects
@@
 			)
 		)
-		(property "Footprint" ""
+		(property "Footprint" "Button_Switch_THT:SW_TH_Tactile_Omron_B3F-100x"
 			(at 64.77 40.64 0)
 			(effects
@@
 			)
 		)
-		(property "Footprint" ""
+		(property "Footprint" "Capacitor_SMD:C_0603_1608Metric"
 			(at 272.7452 35.56 0)
 			(effects
@@
 			)
 		)
-		(property "Footprint" ""
+		(property "Footprint" "Capacitor_SMD:C_0603_1608Metric"
 			(at 153.3652 49.53 0)
 			(effects
@@
 			)
 		)
-		(property "Footprint" ""
+		(property "Footprint" "Resistor_SMD:R_0603_1608Metric"
 			(at 191.77 116.332 90)
 			(effects
